File: Design/interferometer.kicad_pcb (KiCad board)
At the start: 4 copper layers, 56.9 x 53.3 mm, 42 parts, among them Q1 FDC637BNZ, U1 ADN8810ACPZ, U2 OPA320SAIDBVT, U3 ADR292GRUZ

Commit message: finalise layout
Parts:
- added J1: GS2, Connectors:GS2, F.Cu at (162.3, 89.9)
- moved D2 0.91 mm to (145.8, 111.4)
Routing:
- net Net-(C7-Pad2): track 10.4 -> 29.8 mm
- net /AVSS: track 29.3 -> 25.6 mm, vias 12 -> 8
- net Earth: track 41.1 -> 42.2 mm, vias 16 -> 17
- net /chip_addr0: track 47.9 -> 48.9 mm
- net Net-(D2-Pad1): track 2.40 -> 3.32 mm
- net /chip_addr1: track 45.9 -> 46.8 mm
- net /PD: track 10.0 -> 9.38 mm
- net /RSN: track 8.76 -> 9.30 mm
