File: Design/interferometer.kicad_pcb (KiCad board)
At the start: 4 copper layers, 56.9 x 53.3 mm, 43 parts, among them J1 GS2, Q1 FDC637BNZ, U1 ADN8810ACPZ, U2 OPA320SAIDBVT, U3 ADR292GRUZ

Commit message: Cleanup
Parts:
- removed G***: LOGO, footprints:Alois_name_logo

Commit message: Cleanup
Parts:
- J1: footprint Connectors:GS2 -> Legacy_Connectors:GS2
- Q1, U2: footprint TO_SOT_Packages_SMD:SOT-23-6 -> Package_TO_SOT_SMD:SOT-23-6
Changed lines of the file:
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@@
     (add_net /AVSS)
   )
-  (module Connectors:GS2 (layer F.Cu)
+  (module Legacy_Connectors:GS2 (layer F.Cu)
     (at 162.2756 89.916 270)
     (descr "2-pin solder bridge")
@@
       (effects (font (size 1 1) (thickness 0.15)))
     )
+    (fp_line (start -0.89 -1.27) (end 0.89 -1.27) (layer F.SilkS) (width 0.12))
+    (fp_line (start 0.89 1.27) (end -0.89 1.27) (layer F.SilkS) (width 0.12))
+    (fp_line (start 0.89 1.27) (end 0.89 -1.27) (layer F.SilkS) (width 0.12))
+    (fp_line (start -0.89 -1.27) (end -0.89 1.27) (layer F.SilkS) (width 0.12))
+    (fp_line (start -1.1 -1.45) (end 1.1 -1.45) (layer F.CrtYd) (width 0.05))
+    (fp_line (start -1.1 1.5) (end -1.1 -1.45) (layer F.CrtYd) (width 0.05))
+    (fp_line (start 1.1 1.5) (end -1.1 1.5) (layer F.CrtYd) (width 0.05))
     (fp_line (start 1.1 -1.45) (end 1.1 1.5) (layer F.CrtYd) (width 0.05))
-    (fp_line (start 1.1 1.5) (end -1.1 1.5) (layer F.CrtYd) (width 0.05))
-    (fp_line (start -1.1 1.5) (end -1.1 -1.45) (layer F.CrtYd) (width 0.05))
-    (fp_line (start -1.1 -1.45) (end 1.1 -1.45) (layer F.CrtYd) (width 0.05))
-    (fp_line (start -0.89 -1.27) (end -0.89 1.27) (layer F.SilkS) (width 0.12))
-    (fp_line (start 0.89 1.27) (end 0.89 -1.27) (layer F.SilkS) (width 0.12))
-    (fp_line (start 0.89 1.27) (end -0.89 1.27) (layer F.SilkS) (width 0.12))
-    (fp_line (start -0.89 -1.27) (end 0.89 -1.27) (layer F.SilkS) (width 0.12))
+    (pad 2 smd rect (at 0 0.64 270) (size 1.27 0.97) (layers F.Cu F.Paste F.Mask)
+      (net 8 Earth))
     (pad 1 smd rect (at 0 -0.64 270) (size 1.27 0.97) (layers F.Cu F.Paste F.Mask)
       (net 41 /AVSS))
-    (pad 2 smd rect (at 0 0.64 270) (size 1.27 0.97) (layers F.Cu F.Paste F.Mask)
-      (net 8 Earth))
   )
   (module ADN8810ACPZ:ADR292GRUZ (layer F.Cu)
@@
     )
   )
-  (module TO_SOT_Packages_SMD:SOT-23-6 (layer F.Cu)
+  (module Package_TO_SOT_SMD:SOT-23-6 (layer F.Cu)
     (at 146.05 95.631)
     (descr "6-pin SOT-23 package")
     (tags SOT-23-6)
     (attr smd)
-    (fp_text reference U2 (at 2.667 -0.127 90) (layer F.SilkS)
+    (fp_text reference U2 (at 0 -2.9) (layer F.SilkS)
       (effects (font (size 1 1) (thickness 0.15)))
     )
@@
       (effects (font (size 1 1) (thickness 0.15)))
     )
-    (fp_line (start 0.9 -1.55) (end 0.9 1.55) (layer F.Fab) (width 0.15))
-    (fp_line (start 0.9 1.55) (end -0.9 1.55) (layer F.Fab) (width 0.15))
-    (fp_line (start -0.9 -1.55) (end -0.9 1.55) (layer F.Fab) (width 0.15))
-    (fp_line (start 0.9 -1.55) (end -0.9 -1.55) (layer F.Fab) (width 0.15))
+    (fp_line (start 0.9 -1.55) (end 0.9 1.55) (layer F.Fab) (width 0.1))
+    (fp_line (start 0.9 1.55) (end -0.9 1.55) (layer F.Fab) (width 0.1))
+    (fp_line (start -0.9 -0.9) (end -0.9 1.55) (layer F.Fab) (width 0.1))
+    (fp_line (start 0.9 -1.55) (end -0.25 -1.55) (layer F.Fab) (width 0.1))
+    (fp_line (start -0.9 -0.9) (end -0.25 -1.55) (layer F.Fab) (width 0.1))
     (fp_line (start -1.9 -1.8) (end -1.9 1.8) (layer F.CrtYd) (width 0.05))
     (fp_line (start -1.9 1.8) (end 1.9 1.8) (layer F.CrtYd) (width 0.05))
@@
     (fp_line (start 0.9 -1.61) (end -1.55 -1.61) (layer F.SilkS) (width 0.12))
     (fp_line (start -0.9 1.61) (end 0.9 1.61) (layer F.SilkS) (width 0.12))
+    (fp_text user %R (at 0 0 90) (layer F.Fab)
+      (effects (font (size 0.5 0.5) (thickness 0.075)))
+    )
     (pad 5 smd rect (at 1.1 0) (size 1.06 0.65) (layers F.Cu F.Paste F.Mask)
       (net 19 /~SHDN))
@@
     (pad 1 smd rect (at -1.1 -0.95) (size 1.06 0.65) (layers F.Cu F.Paste F.Mask)
       (net 61 "Net-(C12-Pad1)"))
-    (model packages3d/TO_SOT_Packages_SMD.3dshapes/SOT-23-6.step
+    (model ${KISYS3DMOD}/Package_TO_SOT_SMD.3dshapes/SOT-23-6.wrl
       (at (xyz 0 0 0))
       (scale (xyz 1 1 1))
@@
     )
   )
-  (module TO_SOT_Packages_SMD:SOT-23-6 (layer F.Cu)
+  (module Package_TO_SOT_SMD:SOT-23-6 (layer F.Cu)
     (at 158.158 102.301 90)
     (descr "6-pin SOT-23 package")
@@
       (effects (font (size 1 1) (thickness 0.15)))
     )
-    (fp_line (start 0.9 -1.55) (end 0.9 1.55) (layer F.Fab) (width 0.15))
-    (fp_line (start 0.9 1.55) (end -0.9 1.55) (layer F.Fab) (width 0.15))
-    (fp_line (start -0.9 -1.55) (end -0.9 1.55) (layer F.Fab) (width 0.15))
-    (fp_line (start 0.9 -1.55) (end -0.9 -1.55) (layer F.Fab) (width 0.15))
+    (fp_line (start 0.9 -1.55) (end 0.9 1.55) (layer F.Fab) (width 0.1))
+    (fp_line (start 0.9 1.55) (end -0.9 1.55) (layer F.Fab) (width 0.1))
+    (fp_line (start -0.9 -0.9) (end -0.9 1.55) (layer F.Fab) (width 0.1))
+    (fp_line (start 0.9 -1.55) (end -0.25 -1.55) (layer F.Fab) (width 0.1))
+    (fp_line (start -0.9 -0.9) (end -0.25 -1.55) (layer F.Fab) (width 0.1))
     (fp_line (start -1.9 -1.8) (end -1.9 1.8) (layer F.CrtYd) (width 0.05))
     (fp_line (start -1.9 1.8) (end 1.9 1.8) (layer F.CrtYd) (width 0.05))
@@
     (fp_line (start 0.9 -1.61) (end -1.55 -1.61) (layer F.SilkS) (width 0.12))
     (fp_line (start -0.9 1.61) (end 0.9 1.61) (layer F.SilkS) (width 0.12))
+    (fp_text user %R (at 0 0) (layer F.Fab)
+      (effects (font (size 0.5 0.5) (thickness 0.075)))
+    )
     (pad 5 smd rect (at 1.1 0 90) (size 1.06 0.65) (layers F.Cu F.Paste F.Mask)
       (net 44 "Net-(Q1-Pad5)"))
@@
     (pad 1 smd rect (at -1.1 -0.95 90) (size 1.06 0.65) (layers F.Cu F.Paste F.Mask)
       (net 49 "Net-(Q1-Pad1)"))
-    (model packages3d/TO_SOT_Packages_SMD.3dshapes/SOT-23-6.step
-      (at (xyz 0 0 0))
-      (scale (xyz 1 1 1))
+    (model ${KISYS3DMOD}/Package_TO_SOT_SMD.3dshapes/SOT-23-6.wrl
+      (at (xyz 0 0 0))
+      (scale (xyz 1 1 1))
