File: Design/interferometer.sch (KiCad schematic (older format))
At the start: 42 parts, among them J1 GS2, Q1 FDC637BNZ, U1 ADN8810ACPZ, U2 OPA320SAIDBVT, U3 ADR292GRUZ

Commit message: Cleanup
Parts:
- R1: value 680k -> 680k ohm 1%
- R10: value 100R -> 100 ohm
- R11: value 5.1k -> 5.1k ohm
- R2: value 21k -> 21k ohm 1%
- R3: value 66.5R -> 66.5 ohm 0.1%
- R4: value 7.87k -> 7.87k ohm
- R5, R6, R7, R8: value 100k -> 100k ohm
- R9: value 220R -> 220 ohm
Changed lines of the file:
@@
 P 7230 4820
 F 0 "R3" H 7000 4890 50  0000 L CNN
-F 1 "66.5R" H 6950 4790 50  0000 L CNN
+F 1 "66.5 ohm 0.1%" H 6950 4790 50  0000 L CNN
 F 2 "Resistors_SMD:R_0805" V 7160 4820 50  0001 C CNN
 F 3 "" H 7230 4820 50  0001 C CNN
@@
 P 8650 3750
 F 0 "R1" H 8700 3900 50  0000 L CNN
-F 1 "680k" H 8700 3800 50  0000 L CNN
+F 1 "680k ohm 1%" H 8700 3800 50  0000 L CNN
 F 2 "Resistors_SMD:R_0805" V 8580 3750 50  0001 C CNN
 F 3 "" H 8650 3750 50  0001 C CNN
@@
 P 8950 4000
 F 0 "R2" V 8950 4000 50  0000 C CNN
-F 1 "21k" V 8834 4000 50  0000 C CNN
+F 1 "21k ohm 1%" V 8834 4000 50  0000 C CNN
 F 2 "Resistors_SMD:R_0805" V 8880 4000 50  0001 C CNN
 F 3 "" H 8950 4000 50  0001 C CNN
@@
 P 9250 5200
 F 0 "R4" V 9250 5200 50  0000 C CNN
-F 1 "7.87k" V 9350 5200 50  0000 C CNN
+F 1 "7.87k ohm" V 9350 5200 50  0000 C CNN
 F 2 "Resistors_SMD:R_0805" V 9180 5200 50  0001 C CNN
 F 3 "" H 9250 5200 50  0001 C CNN
@@
 P 10550 4550
 F 0 "R8" H 10620 4596 50  0000 L CNN
-F 1 "100k" H 10620 4505 50  0000 L CNN
+F 1 "100k ohm" H 10620 4505 50  0000 L CNN
 F 2 "Resistors_SMD:R_0805_HandSoldering" V 10480 4550 50  0001 C CNN
 F 3 "" H 10550 4550 50  0001 C CNN
@@
 P 8200 2750
 F 0 "R7" H 8270 2796 50  0000 L CNN
-F 1 "100k" H 8270 2705 50  0000 L CNN
+F 1 "100k ohm" H 8270 2705 50  0000 L CNN
 F 2 "Resistors_SMD:R_0805_HandSoldering" V 8130 2750 50  0001 C CNN
 F 3 "" H 8200 2750 50  0001 C CNN
@@
 P 6900 1800
 F 0 "R6" H 6970 1846 50  0000 L CNN
-F 1 "100k" H 6970 1755 50  0000 L CNN
+F 1 "100k ohm" H 6970 1755 50  0000 L CNN
 F 2 "Resistors_SMD:R_0805_HandSoldering" V 6830 1800 50  0001 C CNN
 F 3 "" H 6900 1800 50  0001 C CNN
@@
 P 7450 1200
 F 0 "R5" H 7520 1246 50  0000 L CNN
-F 1 "100k" H 7520 1155 50  0000 L CNN
+F 1 "100k ohm" H 7520 1155 50  0000 L CNN
 F 2 "Resistors_SMD:R_0805_HandSoldering" V 7380 1200 50  0001 C CNN
 F 3 "" H 7450 1200 50  0001 C CNN
@@
 P 3300 2650
 F 0 "R9" H 3150 2700 50  0000 L CNN
-F 1 "220R" H 3050 2600 50  0000 L CNN
+F 1 "220 ohm" H 3050 2600 50  0000 L CNN
 F 2 "Resistors_SMD:R_0805_HandSoldering" V 3230 2650 50  0001 C CNN
 F 3 "" H 3300 2650 50  0001 C CNN
@@
 P 3650 2650
 F 0 "R10" H 3450 2700 50  0000 L CNN
-F 1 "100R" H 3400 2600 50  0000 L CNN
+F 1 "100 ohm" H 3400 2600 50  0000 L CNN
 F 2 "Resistors_SMD:R_0805_HandSoldering" V 3580 2650 50  0001 C CNN
 F 3 "" H 3650 2650 50  0001 C CNN
@@
 P 10100 5050
 F 0 "R11" H 10170 5096 50  0000 L CNN
-F 1 "5.1k" H 10170 5005 50  0000 L CNN
+F 1 "5.1k ohm" H 10170 5005 50  0000 L CNN
 F 2 "Resistors_SMD:R_0805_HandSoldering" V 10030 5050 50  0001 C CNN
 F 3 "" H 10100 5050 50  0001 C CNN
