File: pcb/interferometer.kicad_pcb (KiCad board)
At the start: 4 copper layers, 56.9 x 53.3 mm, 43 parts, among them J1 GS2, Q1 FDC637BNZ, U1 ADN8810ACPZ, U2 OPA320SAIDBVT, U3 ADR292GRUZ

Commit message: Board updated by fiverr.com:Saqibchaudhr141
Parts:
- removed G***: LOGO, footprints:Alois_name_logo
- C1, C11, C12, C13, C14, C2, C3, C4, C5, C6, C7: footprint Capacitors_SMD:C_0805_HandSoldering -> Capacitor_SMD:C_0603_1608Metric
- C10, C8, C9: footprint Capacitors_SMD:C_1210_HandSoldering -> Capacitor_SMD:C_0603_1608Metric
- D1, D2: footprint LEDs:LED_0805 -> LED_SMD:LED_0805_2012Metric_Castellated
- J1: footprint Connectors:GS2 -> 1x02 GS2:GS2
- Q1, U2: footprint TO_SOT_Packages_SMD:SOT-23-6 -> OPA320SAIDBVT:SOT95P280X145-6N
- R1, R2, R3, R4: footprint Resistors_SMD:R_0805 -> Resistor_SMD:R_0805_2012Metric
- R10, R11, R5, R6, R7, R8, R9: footprint Resistors_SMD:R_0805_HandSoldering -> Resistor_SMD:R_0805_2012Metric
- TP1, TP2, TP3, TP4: footprint Measurement_Points:Measurement_Point_Round-SMD-Pad_Small -> TestPoint:TestPoint_Pad_D1.5mm
- moved TP2 7.24 mm to (166.8, 82.9)
- moved J1 6.84 mm to (162.8, 83.1), turned to 180 degrees
- moved TP1 5.05 mm to (172.0, 116.3)
- moved C10 1.26 mm to (154.9, 116.2)
- moved C9 1.15 mm to (150.5, 116.2)
- moved R1 0.68 mm to (141.8, 96.5)
- moved R10 0.42 mm to (145.8, 117.5)
- moved Q1 0.20 mm to (158.0, 102.4)
- moved TP4 0.18 mm to (146.1, 107.7)
- moved U2 0.08 mm to (146.1, 95.5)
Routing:
- net Earth: track 39.9 -> 223.5 mm, vias 17 -> 13
- net /AVSS: track 26.7 -> 118.4 mm, vias 12 -> 11
- net /3v3: track 15.6 -> 96.6 mm, vias 8 -> 3
- net /5v: track 26.1 -> 86.0 mm, vias 8 -> 3
- net Net-(C3-Pad1): track 59.4 -> 47.9 mm, vias 0 -> 1
- net /A0: track 21.2 -> 31.4 mm
- net /4.096_VREF: track 11.0 -> 18.7 mm
- net Net-(D2-Pad1): track 3.32 -> 7.60 mm
- net /~CS: track 28.4 -> 32.6 mm, vias 2 -> 1
- net /SCK: track 30.6 -> 33.7 mm, vias 2 -> 1
- net Net-(C7-Pad2): track 30.9 -> 28.2 mm
- net /LD: track 12.0 -> 9.46 mm, vias 0 -> 1
- net /MOSI: track 31.7 -> 29.3 mm, vias 2 -> 1
- net Net-(C12-Pad1): track 29.1 -> 31.1 mm
- net /~laser_standby: track 38.0 -> 39.6 mm
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- added copper zone on F.Cu, net /5v
- added copper zone on B.Cu, net Earth
- removed copper zone on PVDD-DVDD, net /3v3
- removed copper zone on PVDD-DVDD, net /5v
- removed copper zone on VSS-GND, net /AVSS
- removed copper zone on VSS-GND, net Earth
Other:
- copper layers 4 -> 2
