File: pcb/interferometer.sch (KiCad schematic (older format))
At the start: 42 parts, among them J1 GS2, Q1 FDC637BNZ, U1 ADN8810ACPZ, U2 OPA320SAIDBVT, U3 ADR292GRUZ

Commit message: Board updated by fiverr.com:Saqibchaudhr141
Parts:
- removed U1: ADN8810ACPZ, ADN8810ACPZ:ADN8810ACPZ, symbol ADN8810ACPZ:ADN8810ACP
- removed U2: OPA320SAIDBVT, TO_SOT_Packages_SMD:SOT-23-6, symbol ADN8810ACPZ:OPA320SAIDBVT
- added U1: ADN8810ACP, ADN8810ACPZ:ADN8810ACPZ, symbol interferometer-rescue:ADN8810ACP
- added U2: OPA320SAIDBVT, OPA320SAIDBVT:SOT95P280X145-6N, symbol OPA320SAIDBVT:OPA320SAIDBVT
- C1, C11, C13, C14, C2, C3, C4, C5, C6, C7: value 0.1uF -> 100nF; footprint Capacitors_SMD:C_0805_HandSoldering -> Capacitor_SMD:C_0805_2012Metric_Pad1.15x1.40mm_HandSolder; Manufacturer_Name (none) -> Samsung Electro-Mechanics; Manufacturer_Part_Number (none) -> CL21B104JBCNNNC; manf# (none) -> CL21B104JBCNNNC
- C10, C8, C9: footprint Capacitors_SMD:C_1210_HandSoldering -> Capacitor_SMD:C_1210_3225Metric_Pad1.42x2.65mm_HandSolder
- C12: footprint Capacitors_SMD:C_0805_HandSoldering -> Capacitor_SMD:C_0805_2012Metric_Pad1.15x1.40mm_HandSolder; Manufacturer_Name (none) -> Samsung Electro-Mechanics; Manufacturer_Part_Number (none) -> CL21C820JBANNNC; manf# (none) -> CL21C820JBANNNC
- D1, D2: value LED -> LED GREEN; footprint LEDs:LED_0805 -> LED_SMD:LED_0805_2012Metric; Manufacturer_Name (none) -> Lite-On; Manufacturer_Part_Number (none) -> LTST-C171KGKT; manf# (none) -> LTST-C171KGKT
- J1: footprint Connectors:GS2 -> 1x02 GS2:GS2
- LD1: value Laserdiode_N_TYPE -> Laserdiode_N_TYPE (2.2-2.5v); Farnell SC12525 -> (none); Manufacturer_Name (none) -> LASER COMPONENTS; Manufacturer_Part_Number (none) -> ADL-65055TL; manufacturer LASER COMPONENTS -> (none)
- Q1: footprint TO_SOT_Packages_SMD:SOT-23-6 -> OPA320SAIDBVT:SOT95P280X145-6N; symbol ADN8810ACPZ:FDC637BNZ -> interferometer-rescue:FDC637BNZ; Digikey FDC637BNZCT-ND -> (none); Manufacturer_Name (none) -> ON Semiconductor; Manufacturer_Part_Number (none) -> FDC637BNZ; Mouser 512-FDC637BNZ -> (none); Mouser Part Number (none) -> 512-FDC637BNZ; manufacturer ON Semiconductor -> (none)
- R1: value 680k -> 680kohms; footprint Resistors_SMD:R_0805 -> Resistor_SMD:R_0805_2012Metric
- R10: value 100R -> 100ohms; footprint Resistors_SMD:R_0805_HandSoldering -> Resistor_SMD:R_0805_2012Metric_Pad1.15x1.40mm_HandSolder
- R11: value 5.1k -> 5.1kohms; footprint Resistors_SMD:R_0805_HandSoldering -> Resistor_SMD:R_0805_2012Metric
- R2: value 21k -> 21Kohms; footprint Resistors_SMD:R_0805 -> Resistor_SMD:R_0805_2012Metric
- R3: value 66.5R -> 66.5ohms; footprint Resistors_SMD:R_0805 -> Resistor_SMD:R_0805_2012Metric; Manufacturer_Name (none) -> Panasonic; Manufacturer_Part_Number (none) -> ERJ-6ENF66R5V; manf# (none) -> ERJ-6ENF66R5V
- R4: value 7.87k -> 7.87kohms; footprint Resistors_SMD:R_0805 -> Resistor_SMD:R_0805_2012Metric
- R5, R6, R7, R8: value 100k -> 100kohms; footprint Resistors_SMD:R_0805_HandSoldering -> Resistor_SMD:R_0805_2012Metric_Pad1.15x1.40mm_HandSolder; Digikey P100KDATR-ND -> (none); Farnell 1577686 -> (none); Manufacturer_Name (none) -> Panasonic; Manufacturer_Part_Number (none) -> ERA-6AEB104V; Mouser 667-ERA-6AEB104V -> (none); manufacturer Panasonic -> (none)
- R9: value 220R -> 220ohms; footprint Resistors_SMD:R_0805_HandSoldering -> Resistor_SMD:R_0805_2012Metric_Pad1.15x1.40mm_HandSolder
- SHIELD1: symbol freetronics_schematic:ARDUINO_SHIELD -> interferometer-rescue:ARDUINO_SHIELD
- TP1, TP2, TP3, TP4: footprint Measurement_Points:Measurement_Point_Round-SMD-Pad_Small -> TestPoint:TestPoint_Pad_D1.5mm; symbol freetronics_schematic:TESTPOINT -> interferometer-rescue:TESTPOINT
- U3: symbol ADN8810ACPZ:ADR292GRUZ -> interferometer-rescue:ADR292GRUZ; Digikey ADR292GRUZ-ND -> (none); Manufacturer_Name (none) -> Analog Devices; Manufacturer_Part_Number (none) -> ADR292GRUZ; Mouser 584-ADR292GRUZ -> (none); Mouser Part Number (none) -> 584-ADR292GRUZ; manufacturer Analog Devices -> (none)
Connections:
- net 3v3: now also U2.6 (V+)
- net 4.096_VREF: now also U1.14 (VREF)
- net 5v: now also U1.15 (AVDD), U1.23 (DVDD)
- net AVSS: now also U1.12 (ENCOMP), U1.16 (AVSS), U1.18 (DVSS), U1.25 (EPAD), U2.2 (V-)
- net Earth: now also U1.24 (DGND)
- net IOUT: now also U1.10 (IOUT)
- net MOSI: now also U1.19 (SDI)
- net PD: now also U2.4 (-IN)
- net RSN: now also U1.2 (RSN)
- net SCK: now also U1.20 (SCLK)
- net chip_addr0: now also U1.5 (ADDR0)
- net chip_addr1: now also U1.4 (ADDR1)
- net chip_addr2: now also U1.1 (ADDR2)
- net ~CS: now also U1.21 (~CS)
- net ~SHDN: now also U2.5 (~SHDN)
- net ~laser_reset: now also U1.22 (~RESET)
- net ~laser_standby: now also U1.7 (~SB)
- net at C3.1, JP1.2: now also U1.11 (PVDD), U1.8 (PVDD)
- net at C12.1, C14.2, R4.1: now also U2.1 (VOUT)
- net at C7.2, R1.2, R2.2: now also U2.3 (+IN)
