File: pcb/interferometer.sch (KiCad schematic (older format))
At the start: 42 parts, among them J1 GS2, Q1 FDC637BNZ, U1 ADN8810ACPZ, U2 OPA320SAIDBVT, U3 ADR292GRUZ

Commit message: Cleanup. Add spice models.
Parts:
- C1, C10, C11, C12, C13, C14, C2, C3, C4, C5, C6, C7, C8, C9: symbol Device:C -> interferometer-rescue:C-Device
- D1, D2: symbol Device:LED -> interferometer-rescue:LED-Device
- JP1, JP2, JP3, JP4: symbol Device:Jumper_NC_Dual -> interferometer-rescue:Jumper_NC_Dual-Device
- LD1: symbol Device:Laserdiode_N_TYPE -> interferometer-rescue:Laserdiode_N_TYPE-Device
- R1, R10, R11, R2, R3, R4, R5, R6, R7, R8, R9: symbol Device:R -> interferometer-rescue:R-Device
Changed lines of the file:
@@
 $EndDescr
 $Comp
-L Device:Laserdiode_N_TYPE LD1
+L interferometer-rescue:Laserdiode_N_TYPE-Device LD1
 U 1 1 5919F1C9
 P 1900 1715
@@
 GND
 $Comp
-L power:GNDA #PWR01
+L interferometer-rescue:GNDA-power #PWR01
 U 1 1 591C35DD
 P 2250 4350
@@
 Analog and digital grounds
 $Comp
-L Device:C C1
+L interferometer-rescue:C-Device C1
 U 1 1 591C3B82
 P 8750 850
@@
 4.096v voltage reference
 $Comp
-L power:Earth #PWR02
+L interferometer-rescue:Earth-power #PWR02
 U 1 1 591C415F
 P 2650 4350
@@
 AVSS
 $Comp
-L Device:C C8
+L interferometer-rescue:C-Device C8
 U 1 1 591C4360
 P 1150 4200
@@
 $EndComp
 $Comp
-L power:GNDA #PWR03
+L interferometer-rescue:GNDA-power #PWR03
 U 1 1 591C43D1
 P 1150 4350
@@
 $EndComp
 $Comp
-L Device:C C3
+L interferometer-rescue:C-Device C3
 U 1 1 591C4BB6
 P 10200 1100
@@
 5v
 $Comp
-L power:Earth #PWR04
+L interferometer-rescue:Earth-power #PWR04
 U 1 1 591C5737
 P 9650 2800
@@
 Laser driver address jumpers
 $Comp
-L Device:Jumper_NC_Dual JP4
+L interferometer-rescue:Jumper_NC_Dual-Device JP4
 U 1 1 591C6801
 P 5350 3950
@@
 $EndComp
 $Comp
-L Device:Jumper_NC_Dual JP2
+L interferometer-rescue:Jumper_NC_Dual-Device JP2
 U 1 1 591C6851
 P 3750 3950
@@
 $EndComp
 $Comp
-L Device:Jumper_NC_Dual JP3
+L interferometer-rescue:Jumper_NC_Dual-Device JP3
 U 1 1 591C689D
 P 4550 3950
@@
 ADDR2
 $Comp
-L Device:C C4
+L interferometer-rescue:C-Device C4
 U 1 1 591C8F57
 P 7350 1600
@@
 Power supplies and low frequency filtering
 $Comp
-L Device:C C6
+L interferometer-rescue:C-Device C6
 U 1 1 591CA8F6
 P 9150 2950
@@
 $EndComp
 $Comp
-L power:GNDA #PWR05
+L interferometer-rescue:GNDA-power #PWR05
 U 1 1 591CAC9F
 P 9150 3150
@@
 AVSS
 $Comp
-L power:Earth #PWR06
+L interferometer-rescue:Earth-power #PWR06
 U 1 1 591CC522
 P 3750 4250
@@
 $EndComp
 $Comp
-L power:Earth #PWR07
+L interferometer-rescue:Earth-power #PWR07
 U 1 1 591CC620
 P 4550 4250
@@
 $EndComp
 $Comp
-L power:Earth #PWR08
+L interferometer-rescue:Earth-power #PWR08
 U 1 1 591CC6E3
 P 5350 4250
@@
 $EndComp
 $Comp
-L power:GNDA #PWR09
+L interferometer-rescue:GNDA-power #PWR09
 U 1 1 591CD640
 P 7350 1850
@@
 $EndComp
 $Comp
-L Device:C C9
+L interferometer-rescue:C-Device C9
 U 1 1 591CDD86
 P 1050 5550
@@
 $EndComp
 $Comp
-L power:GNDA #PWR010
+L interferometer-rescue:GNDA-power #PWR010
 U 1 1 591CE000
 P 1050 5800
@@
 LD
 $Comp
-L Device:R R3
+L interferometer-rescue:R-Device R3
 U 1 1 591CE293
 P 7230 4820
@@
 $EndComp
 $Comp
-L Device:C C11
+L interferometer-rescue:C-Device C11
 U 1 1 591CF24A
 P 3405 5530
@@
 3v3
 $Comp
-L Device:C C10
+L interferometer-rescue:C-Device C10
 U 1 1 591D633E
 P 2450 5550
@@
 $EndComp
 $Comp
-L power:GNDA #PWR011
+L interferometer-rescue:GNDA-power #PWR011
 U 1 1 591D6345
 P 2450 5800
@@
 AVSS
 $Comp
-L Device:C C2
+L interferometer-rescue:C-Device C2
 U 1 1 591D6A0E
 P 8300 900
@@
 AVSS
 $Comp
-L Device:Jumper_NC_Dual JP1
+L interferometer-rescue:Jumper_NC_Dual-Device JP1
 U 1 1 591D7A74
 P 10585 900
@@
 3v3
 $Comp
-L Device:C C5
+L interferometer-rescue:C-Device C5
 U 1 1 591D8E08
 P 1450 1700
@@
 AVSS
 $Comp
-L power:Earth #PWR012
+L interferometer-rescue:Earth-power #PWR012
 U 1 1 591D7D5F
 P 8300 1100
@@
 AVSS
 $Comp
-L Device:R R1
+L interferometer-rescue:R-Device R1
 U 1 1 591DF768
 P 8650 3750
@@
 $EndComp
 $Comp
-L Device:R R2
+L interferometer-rescue:R-Device R2
 U 1 1 591DF87A
 P 8950 4000
@@
 3v3
 $Comp
-L Device:C C7
+L interferometer-rescue:C-Device C7
 U 1 1 591DFDB3
 P 8350 3750
@@
 PD
 $Comp
-L Device:R R4
+L interferometer-rescue:R-Device R4
 U 1 1 591E038E
 P 9250 5200
@@
 $EndComp
 $Comp
-L Device:C C12
+L interferometer-rescue:C-Device C12
 U 1 1 591E07E5
 P 9250 5600
@@
 NoConn ~ 7080 3815
 $Comp
-L Device:R R8
+L interferometer-rescue:R-Device R8
 U 1 1 591DD952
 P 10550 4550
@@
 3v3
 $Comp
-L Device:R R7
+L interferometer-rescue:R-Device R7
 U 1 1 591DE4AD
 P 8200 2750
@@
 3v3
 $Comp
-L Device:R R6
+L interferometer-rescue:R-Device R6
 U 1 1 591DEC98
 P 6900 1800
@@
 3v3
 $Comp
-L Device:R R5
+L interferometer-rescue:R-Device R5
 U 1 1 591DF4B3
 P 7450 1200
@@
 NoConn ~ 4300 3100
 $Comp
-L Device:LED D1
+L interferometer-rescue:LED-Device D1
 U 1 1 591E6733
 P 3300 2250
@@
 $EndComp
 $Comp
-L Device:R R9
+L interferometer-rescue:R-Device R9
 U 1 1 591E706A
 P 3300 2650
@@
 $EndComp
 $Comp
-L power:GNDA #PWR013
+L interferometer-rescue:GNDA-power #PWR013
 U 1 1 591E7828
 P 3300 2850
@@
 $EndComp
 $Comp
-L Device:LED D2
+L interferometer-rescue:LED-Device D2
 U 1 1 591E8C37
 P 3650 2350
@@
 $EndComp
 $Comp
-L Device:R R10
+L interferometer-rescue:R-Device R10
 U 1 1 591E93EB
 P 3650 2650
@@
 $EndComp
 $Comp
-L power:GNDA #PWR014
+L interferometer-rescue:GNDA-power #PWR014
 U 1 1 591E9451
 P 3650 2850
@@
 A0
 $Comp
-L power:GNDA #PWR015
+L interferometer-rescue:GNDA-power #PWR015
 U 1 1 591F4592
 P 10200 1350
@@
 	8750 1100 8750 1000
 $Comp
-L power:GNDA #PWR016
+L interferometer-rescue:GNDA-power #PWR016
 U 1 1 591F4F47
 P 8750 1100
@@
 $EndComp
 $Comp
-L power:GNDA #PWR017
+L interferometer-rescue:GNDA-power #PWR017
 U 1 1 591F5F82
 P 3405 5790
@@
 	3405 5790 3405 5680
 $Comp
-L Device:C C13
+L interferometer-rescue:C-Device C13
 U 1 1 592057BF
 P 8500 5150
@@
 Connection ~ 9100 5000
 $Comp
-L power:GNDA #PWR018
+L interferometer-rescue:GNDA-power #PWR018
 U 1 1 59205C76
 P 8500 5350
@@
 	7850 3500 7850 3650
 $Comp
-L power:GNDA #PWR019
+L interferometer-rescue:GNDA-power #PWR019
 U 1 1 59206D7C
 P 7850 3650
@@
 $EndComp
 $Comp
-L power:GNDA #PWR020
+L interferometer-rescue:GNDA-power #PWR020
 U 1 1 5920C7C9
 P 1450 2150
@@
 	9500 4600 9700 4600
 $Comp
-L Device:R R11
+L interferometer-rescue:R-Device R11
 U 1 1 592166B5
 P 10100 5050
@@
 $EndComp
 $Comp
-L Device:C C14
+L interferometer-rescue:C-Device C14
 U 1 1 592167F4
 P 9900 4600
@@
 	10050 4600 10100 4600
 $Comp
-L power:GNDA #PWR021
+L interferometer-rescue:GNDA-power #PWR021
 U 1 1 59216D38
 P 10100 5300
@@
 $EndComp
 $Comp
-L power:GNDA #PWR022
+L interferometer-rescue:GNDA-power #PWR022
 U 1 1 5921A1DD
 P 1550 7050
